File: bldc_motor_cntroller/io_interface.sch (KiCad schematic (older format))
At the start: 0 parts

Commit message: schematic annotation. added bulk caps. moved shunt res to powersheet.
Signed-off-by: azmat bilal <azmat.bilal@outlook.com>
Parts:
- added C1, C2, C3, C4, C5: 82pF, symbol Device:C_Small
- added C6: 100nF, symbol Device:C_Small
- added J1: SM06B-SRSS-TB, Connector_JST:JST_SH_SM06B-SRSS-TB_1x06-1MP_P1.00mm_Horizontal, symbol Connector_Generic:Conn_01x06
- added J2: GENERIC 2.54P 06, Connector_PinHeader_2.54mm:PinHeader_1x06_P2.54mm_Horizontal, symbol Connector_Generic:Conn_01x06
- added J3: Conn_01x10, symbol Connector_Generic:Conn_01x10
- added J4: Conn_01x05, symbol Connector_Generic:Conn_01x05
- added J5: USB_B_Micro, symbol Connector:USB_B_Micro
- added J6: TC2030 Tag-connect, Connector:Tag-Connect_TC2030-IDC-NL_2x03_P1.27mm_Vertical, symbol Connector_Generic:Conn_02x03_Odd_Even
- added J7: SH-SM02B-SRSS, Connector_JST:JST_SH_SM02B-SRSS-TB_1x02-1MP_P1.00mm_Horizontal, symbol Connector_Generic:Conn_01x02
- added R1, R2, R6, R7, R8: 0R, symbol Device:R
- added R10, R9: 22R, symbol Device:R
- added R11: 10k, symbol Device:R
- added R12: 120R, symbol Device:R
- added R3, R4, R5: 3.3k, Resistor_SMD:R_0402_1005Metric, symbol Device:R
- added SW1, SW2: SW_Push, symbol Switch:SW_Push
- added TP1, TP2, TP3: TestPoint, symbol Connector:TestPoint
- added U1: TCAN332G, symbol Interface_CAN_LIN:TCAN332G
Connections:
- new net: C1.1, J3.2 (Pin_2), R1.1
- new net: C2.1, J3.3 (Pin_3), R2.1
- new net: C3.1, J3.7 (Pin_7), R6.1
- new net: C4.1, J3.8 (Pin_8), R7.1
- new net: C5.1, J3.9 (Pin_9), R8.1
- new net: J5.2 (D-), R10.2
- new net: J5.3 (D+), R9.2
- new net: J7.2 (Pin_2), R12.1, U1.6 (CANL)
- new net: J7.1 (Pin_1), R12.2, U1.7 (CANH)
- new net +5V: J1.2 (Pin_2), J2.2 (Pin_2)
- new net BOOT0: R11.2, SW1.2
- new net CAN_D: U1.1 (TXD)
- new net CAN_R: U1.4 (RXD)
- new net DEBUG_SWCLK: J4.4 (Pin_4), J6.4 (Pin_4)
- new net DEBUG_SWDIO: J4.2 (Pin_2), J6.2 (Pin_2)
- new net DEBUG_nRESET: J4.3 (Pin_3), J6.3 (Pin_3), SW2.2
- new net ENC_A: J1.3 (Pin_3), J2.3 (Pin_3), R5.2
- new net ENC_B: J1.4 (Pin_4), J2.4 (Pin_4), R4.2
- new net ENC_Z: J1.5 (Pin_5), J2.5 (Pin_5), R3.2
- new net GND: C1.2, C2.2, C3.2, C4.2, C5.2, C6.1, J1.6 (Pin_6), J2.6 (Pin_6), J3.10 (Pin_10), J4.5 (Pin_5), J5.5 (GND), J5.6 (Shield), J6.5 (Pin_5), R11.1, SW2.1, U1.2 (GND)
- new net GPIO_1: R1.2
- new net GPIO_2: R2.2
- new net GPIO_3: J3.4 (Pin_4)
- new net GPIO_4: J3.5 (Pin_5)
- new net GPIO_5: J3.6 (Pin_6)
- new net GPIO_6: R6.2
- new net GPIO_7: R7.2
- new net GPIO_8: R8.2
- new net USB_DM: R10.1, TP3.1
- new net USB_DP: R9.1, TP2.1
- new net VBUS: J5.1 (VBUS), TP1.1
- new net VDD: C6.2, J1.1 (Pin_1), J2.1 (Pin_1), J3.1 (Pin_1), J4.1 (Pin_1), J6.1 (Pin_1), R3.1, R4.1, R5.1, SW1.1, U1.3 (VCC)
- no-connect marks 0 -> 2
Other:
- note added: "DEBUG"
- note added: "DIGITAL COMMUNICATION"
- note added: "ENCODER INTERFACE"
- note added: "Optional RC filter. use 3.3k resistor with \n82pF cap. if unused place a shunt resistor \nand no cap."
- note added: "Side mount JST-SH series connector. its small\nin size and crimped cables are available from \nmajor hobby shops."
