File: bldc_motor_cntroller/peripheral_interface.sch (KiCad schematic (older format))
At the start: 0 parts

Commit message: added braking circuit. added encoder interface.
Signed-off-by: azmat bilal <azmat.bilal@outlook.com>
Parts:
- added C?: 2.2uF 25V, Capacitor_SMD:C_0402_1005Metric, symbol Device:C_Small
- added C?: 100nF 50V, Capacitor_SMD:C_0402_1005Metric, symbol Device:C_Small
- added C?: 2.2uF 16V, Capacitor_SMD:C_0402_1005Metric, symbol Device:C_Small
- added D?: MBR140SFT1G, Diode_SMD:D_SOD-123F, symbol Device:D_Schottky
- added J?: SM06B-SRSS-TB, Connector_JST:JST_SH_SM06B-SRSS-TB_1x06-1MP_P1.00mm_Horizontal, symbol Connector_Generic:Conn_01x06
- added J?: GENERIC 2.54P 06, Connector_PinHeader_2.54mm:PinHeader_1x06_P2.54mm_Horizontal, symbol Connector_Generic:Conn_01x06
- added J?: Terminal_01x02, symbol Connector:Screw_Terminal_01x02
- added Q? (x2): CSD18540Q5B, Package_TO_SOT_SMD:TDSON-8-1, symbol Transistor_FET:CSD18540Q5B
- added R? (x3): 3.3k, Resistor_SMD:R_0402_1005Metric, symbol Device:R
- added R? (x2): 2R2, Capacitor_SMD:C_0402_1005Metric, symbol Device:R
- added R? (x3): 3.3k, symbol Device:R
- added TH?: 10k, Resistor_SMD:R_0402_1005Metric, symbol Device:Thermistor
- added U?: LM5109BSD, Package_SON:WSON-8_4x4mm_P0.8mm, symbol Driver_FET:LM5109BSD
Connections:
- new net: R?.1, U?.5 (LO)
- new net: C?.2, J?.1 (Pin_1), Q?.1 (S), Q?.2 (S), Q?.3 (S), Q?.5 (D), U?.6 (HS)
- new net: R?.1, U?.7 (HO)
- new net: C?.1, D?.1 (K), U?.8 (HB)
- new net: Q?.4 (G), R?.2 (x2)
- new net +5V: J?.2 (Pin_2), J?.2 (Pin_2)
- new net CTRL_HI: R?.2, U?.2 (HI)
- new net CTRL_LI: R?.2, U?.3 (LI)
- new net ENC_A: J?.3 (Pin_3), J?.3 (Pin_3), R?.2
- new net ENC_B: J?.4 (Pin_4), J?.4 (Pin_4), R?.2
- new net ENC_Z: J?.5 (Pin_5), J?.5 (Pin_5), R?.2
- new net GND: C?.2, C?.2, J?.2 (Pin_2), J?.6 (Pin_6), J?.6 (Pin_6), Q?.1 (S), Q?.2 (S), Q?.3 (S), R?.1, R?.1, R?.1, U?.4 (VSS), U?.9 (VSS)
- new net GVDD: C?.1, D?.2 (A), U?.1 (VDD)
- new net TEMP_SENSE: C?.1, R?.2, TH?.2
- new net VDC: Q?.5 (D)
- new net VDD: J?.1 (Pin_1), J?.1 (Pin_1), R?.1, R?.1, R?.1, TH?.1
Other:
- note added: "Side mount JST-SH series connector. its small\nin size and crimped cables are available from \nmajor hobby shops."

Commit message: schematic annotation. added bulk caps. moved shunt res to powersheet.
Signed-off-by: azmat bilal <azmat.bilal@outlook.com>
Parts:
- removed C?: 2.2uF 25V, Capacitor_SMD:C_0402_1005Metric, symbol Device:C_Small
- removed C?: 100nF 50V, Capacitor_SMD:C_0402_1005Metric, symbol Device:C_Small
- removed C?: 2.2uF 16V, Capacitor_SMD:C_0402_1005Metric, symbol Device:C_Small
- removed D?: MBR140SFT1G, Diode_SMD:D_SOD-123F, symbol Device:D_Schottky
- removed J?: SM06B-SRSS-TB, Connector_JST:JST_SH_SM06B-SRSS-TB_1x06-1MP_P1.00mm_Horizontal, symbol Connector_Generic:Conn_01x06
- removed J?: GENERIC 2.54P 06, Connector_PinHeader_2.54mm:PinHeader_1x06_P2.54mm_Horizontal, symbol Connector_Generic:Conn_01x06
- removed J?: Terminal_01x02, symbol Connector:Screw_Terminal_01x02
- removed Q? (x2): CSD18540Q5B, Package_TO_SOT_SMD:TDSON-8-1, symbol Transistor_FET:CSD18540Q5B
- removed R? (x3): 3.3k, Resistor_SMD:R_0402_1005Metric, symbol Device:R
- removed R? (x2): 2R2, Capacitor_SMD:C_0402_1005Metric, symbol Device:R
- removed R? (x3): 3.3k, symbol Device:R
- removed TH?: 10k, Resistor_SMD:R_0402_1005Metric, symbol Device:Thermistor
- removed U?: LM5109BSD, Package_SON:WSON-8_4x4mm_P0.8mm, symbol Driver_FET:LM5109BSD
Other:
- note removed: "Side mount JST-SH series connector. its small\nin size and crimped cables are available from \nmajor hobby shops."
