File: bldc_motor_cntroller/power_management.sch (KiCad schematic (older format))
At the start: 0 parts

Commit message: schematic annotation. added bulk caps. moved shunt res to powersheet.
Signed-off-by: azmat bilal <azmat.bilal@outlook.com>
Parts:
- added C10, C7, C8, C9: 150uF 63V poly, Capacitor_SMD:CP_Elec_10x14.3, symbol Device:CP
- added C11, C12: 10uF 63V, Capacitor_SMD:C_1210_3225Metric, symbol Device:C_Small
- added C13: 0.1uF 100V, Capacitor_SMD:C_0402_1005Metric, symbol Device:C_Small
- added C14: 270pF 50V, Capacitor_SMD:C_0402_1005Metric, symbol Device:C_Small
- added C15: 2.2uF 25V, Capacitor_SMD:C_0402_1005Metric, symbol Device:C_Small
- added C16: 100nF 50V, Capacitor_SMD:C_0402_1005Metric, symbol Device:C_Small
- added C17, C18: 1uF 10V, Capacitor_SMD:C_0402_1005Metric, symbol Device:C_Small
- added C19: 0.1uF 25V, Capacitor_SMD:C_0402_1005Metric, symbol Device:C_Small
- added C20: 2.2uF 16V, Capacitor_SMD:C_0402_1005Metric, symbol Device:C_Small
- added D1: MBR140SFT1G, Diode_SMD:D_SOD-123F, symbol Device:D_Schottky
- added J8, J9: XT60, Connector_AMASS:AMASS_XT60-M_1x02_P7.20mm_Vertical, symbol Connector_Generic:Conn_01x02
- added Q1, Q2: CSD18540Q5B, Package_TO_SOT_SMD:TDSON-8-1, symbol Transistor_FET:CSD18540Q5B
- added R13: 10k, Resistor_SMD:R_0402_1005Metric, symbol Device:R
- added R14: 1k, Resistor_SMD:R_0402_1005Metric, symbol Device:R
- added R15, R18: 2R2, Capacitor_SMD:C_0402_1005Metric, symbol Device:R
- added R16, R17, R19: 3.3k, symbol Device:R
- added TH1: 10k, Resistor_SMD:R_0402_1005Metric, symbol Device:Thermistor
- added U2: TLV75733PDBV, Package_TO_SOT_SMD:SOT-23-5, symbol Regulator_Linear:TLV75733PDBV
- added U3: LM5109BSD, Package_SON:WSON-8_4x4mm_P0.8mm, symbol Driver_FET:LM5109BSD
Connections:
- new net: R18.1, U3.5 (LO)
- new net: C16.2, J9.2 (Pin_2), Q1.1 (S), Q1.2 (S), Q1.3 (S), Q2.5 (D), U3.6 (HS)
- new net: R15.1, U3.7 (HO)
- new net: C16.1, D1.1 (K), U3.8 (HB)
- new net: Q1.4 (G), R15.2
- new net: Q2.4 (G), R18.2
- new net +5V: C17.1, U2.1 (IN), U2.3 (EN)
- new net CTRL_HI: R17.2, U3.2 (HI)
- new net CTRL_LI: R16.2, U3.3 (LI)
- new net GND: C10.2, C11.2, C12.2, C13.2, C14.2, C15.2, C17.2, C18.2, C19.2, C20.2, C7.2, C8.2, C9.2, J8.1 (Pin_1), J9.1 (Pin_1), Q2.1 (S), Q2.2 (S), Q2.3 (S), R14.2, R16.1, R17.1, R19.1, U2.2 (GND), U3.4 (VSS), U3.9 (VSS)
- new net GVDD: C15.1, D1.2 (A), U3.1 (VDD)
- new net TEMP_SENSE: C20.1, R19.2, TH1.2
- new net VBUS_SENSE: C14.1, R13.2, R14.1
- new net VDC: C10.1, C11.1, C12.1, C13.1, C7.1, C8.1, C9.1, J8.2 (Pin_2), Q1.5 (D), R13.1
- new net VDD: C18.1, C19.1, TH1.1, U2.5 (OUT)
Other:
- note added: "BRAKING CIRCUIT"
